File: circuit/analog_section_low_voltage.sch (KiCad schematic (older format))
At the start: 21 parts

Commit message: Update schematic to rev0.2
Parts:
- added K1: Reed Relay DPST NC, Relay_THT:Relay_StandexMeder_DIP_LowProfile, symbol smartevse:Reed_Relay_DPST_NC
- added Q2: Drive Transistor, Package_TO_SOT_THT:TO-92_Inline, symbol Transistor_BJT:2N3904
- added R14: 2.2k, symbol Device:R_Small
- added R17: 22k, symbol Device:R_Small
- gave numbers to parts that had none: 20
Connections:
- net labels added: CP_con, CP_to_relay, PP_con, PP_to_relay
- wire segments 71 -> 88
Other:
- note removed: "Reed Relays!"
Changed lines of the file:
@@
 Title ""
 Date "2020-04-10"
-Rev "0.1"
+Rev "0.2"
 Comp ""
-Comment1 "TODO: Relay circuit for CP & PP lines"
-Comment2 ""
+Comment1 "DONE: Relay circuit for CP & PP lines"
+Comment2 "TODO: Det. Q2, R14, R17, verify relay circuit"
 Comment3 ""
 Comment4 ""
 $EndDescr
 $Comp
-L Connector:Screw_Terminal_01x12 J?
+L Connector:Screw_Terminal_01x12 J2
 U 1 1 5E903CA7
 P 8100 2700
-F 0 "J?" H 8180 2692 50  0000 L CNN
+F 0 "J2" H 8180 2692 50  0000 L CNN
 F 1 "Screw_Terminal_01x12" H 8180 2601 50  0000 L CNN
 F 2 "" H 8100 2700 50  0001 C CNN
@@
 	7800 2400 7800 1950
 $Comp
-L Device:Polyfuse_Small F?
+L Device:Polyfuse_Small F1
 U 1 1 5E90649F
 P 7800 1850
-F 0 "F?" H 7868 1896 50  0000 L CNN
+F 0 "F1" H 7868 1896 50  0000 L CNN
 F 1 "Polyfuse_Small" H 7868 1805 50  0000 L CNN
 F 2 "" H 7850 1650 50  0001 L CNN
@@
 	7800 1750 7800 1150
 $Comp
-L Device:C_Small C?
+L Device:C_Small C20
 U 1 1 5E906C0D
 P 6200 1300
-F 0 "C?" H 6292 1346 50  0000 L CNN
+F 0 "C20" H 6292 1346 50  0000 L CNN
 F 1 "100n" H 6292 1255 50  0000 L CNN
 F 2 "" H 6200 1300 50  0001 C CNN
@@
 	6200 1150 7800 1150
 $Comp
-L Device:Opamp_Dual_Generic U?
+L Device:Opamp_Dual_Generic U11
 U 1 1 5E9126F4
 P 5600 1800
-F 0 "U?" H 5600 1433 50  0000 C CNN
+F 0 "U11" H 5600 1433 50  0000 C CNN
 F 1 "LM7332" H 5600 1524 50  0000 C CNN
 F 2 "" H 5600 1800 50  0001 C CNN
@@
 $EndComp
 $Comp
-L Device:Opamp_Dual_Generic U?
+L Device:Opamp_Dual_Generic U11
 U 2 1 5E913218
 P 5400 2850
-F 0 "U?" H 5400 3217 50  0000 C CNN
+F 0 "U11" H 5400 3217 50  0000 C CNN
 F 1 "LM7332" H 5400 3126 50  0000 C CNN
 F 2 "" H 5400 2850 50  0001 C CNN
@@
 $EndComp
 $Comp
-L Device:Opamp_Dual_Generic U?
+L Device:Opamp_Dual_Generic U12
 U 3 1 5E913947
 P 5800 1800
-F 0 "U?" H 5758 1846 50  0000 L CNN
+F 0 "U12" H 5758 1846 50  0000 L CNN
 F 1 "LM7332_Power_Supply" H 5758 1755 50  0000 L CNN
 F 2 "" H 5800 1800 50  0001 C CNN
@@
 	5700 2150 5700 2200
 $Comp
-L Device:C_Small C?
+L Device:C_Small C18
 U 1 1 5E918D93
 P 6000 2250
-F 0 "C?" H 6092 2296 50  0000 L CNN
+F 0 "C18" H 6092 2296 50  0000 L CNN
 F 1 "100n" H 6092 2205 50  0000 L CNN
 F 2 "" H 6000 2250 50  0001 C CNN
@@
 	5900 1900 6350 1900
 $Comp
-L Device:R_Small R?
+L Device:R_Small R23
 U 1 1 5E91A28A
 P 5950 2850
-F 0 "R?" V 6146 2850 50  0000 C CNN
+F 0 "R23" V 6146 2850 50  0000 C CNN
 F 1 "1K 1%" V 6055 2850 50  0000 C CNN
 F 2 "" H 5950 2850 50  0001 C CNN
@@
 	4650 2350 4650 2950
 $Comp
-L Device:R_Small R?
+L Device:R_Small R18
 U 1 1 5E91B9F4
 P 4650 2250
-F 0 "R?" H 4709 2296 50  0000 L CNN
+F 0 "R18" H 4709 2296 50  0000 L CNN
 F 1 "15K" H 4709 2205 50  0000 L CNN
 F 2 "" H 4650 2250 50  0001 C CNN
@@
 $EndComp
 $Comp
-L Device:R_Small R?
+L Device:R_Small R19
 U 1 1 5E91BDD8
 P 4650 3350
-F 0 "R?" H 4709 3396 50  0000 L CNN
+F 0 "R19" H 4709 3396 50  0000 L CNN
 F 1 "15K" H 4709 3305 50  0000 L CNN
 F 2 "" H 4650 3350 50  0001 C CNN
@@
 	5100 2750 4950 2750
 $Comp
-L Device:R_Small R?
+L Device:R_Small R20
 U 1 1 5E91C99B
 P 4850 2750
-F 0 "R?" V 4654 2750 50  0000 C CNN
+F 0 "R20" V 4654 2750 50  0000 C CNN
 F 1 "15K" V 4745 2750 50  0000 C CNN
 F 2 "" H 4850 2750 50  0001 C CNN
@@
 $EndComp
 $Comp
-L Device:R_Small R?
+L Device:R_Small R16
 U 1 1 5E91EB9F
 P 4250 3350
-F 0 "R?" H 4309 3396 50  0000 L CNN
+F 0 "R16" H 4309 3396 50  0000 L CNN
 F 1 "15K" H 4309 3305 50  0000 L CNN
 F 2 "" H 4250 3350 50  0001 C CNN
@@
 $EndComp
 $Comp
-L Device:R_Small R?
+L Device:R_Small R15
 U 1 1 5E91EE28
 P 4250 2250
-F 0 "R?" H 4309 2296 50  0000 L CNN
+F 0 "R15" H 4309 2296 50  0000 L CNN
 F 1 "10K" H 4309 2205 50  0000 L CNN
 F 2 "" H 4250 2250 50  0001 C CNN
@@
 Connection ~ 5300 1800
 $Comp
-L Device:R_Small R?
+L Device:R_Small R13
 U 1 1 5E923E93
 P 3950 2250
-F 0 "R?" H 4009 2296 50  0000 L CNN
+F 0 "R13" H 4009 2296 50  0000 L CNN
 F 1 "40.2K" H 4009 2205 50  0000 L CNN
 F 2 "" H 3950 2250 50  0001 C CNN
@@
 	3850 3650 4900 3650
 $Comp
-L Device:R_Small R?
+L Device:R_Small R21
 U 1 1 5E933A1B
 P 5200 3650
-F 0 "R?" V 5004 3650 50  0000 C CNN
+F 0 "R21" V 5004 3650 50  0000 C CNN
 F 1 "10K" V 5095 3650 50  0000 C CNN
 F 2 "" H 5200 3650 50  0001 C CNN
@@
 	4900 3650 5100 3650
 $Comp
-L Device:R_Small R?
+L Device:R_Small R22
 U 1 1 5E943018
 P 5600 3500
-F 0 "R?" H 5541 3454 50  0000 R CNN
+F 0 "R22" H 5541 3454 50  0000 R CNN
 F 1 "1K 1%" H 5541 3545 50  0000 R CNN
 F 2 "" H 5600 3500 50  0001 C CNN
@@
 Wire Wire Line
 	5600 3650 5600 3600
-Connection ~ 5600 3650
 Wire Wire Line
 	5450 3300 5600 3300
@@
 Wire Wire Line
 	7800 3300 7800 3650
-Wire Wire Line
-	5600 3650 7800 3650
-Text Label 7600 3650 0    50   ~ 0
-PP
-$Comp
-L Device:C_Small C?
+Text Label 7500 3650 0    50   ~ 0
+PP_con
+$Comp
+L Device:C_Small C19
 U 1 1 5E949D36
 P 6150 3250
-F 0 "C?" H 6242 3296 50  0000 L CNN
+F 0 "C19" H 6242 3296 50  0000 L CNN
 F 1 "270p" H 6242 3205 50  0000 L CNN
 F 2 "" H 6150 3250 50  0001 C CNN
@@
 	5050 4200 4900 4200
 $Comp
-L Diode:BAT54S D?
+L Diode:BAT54S D5
 U 1 1 5E93ED73
 P 5250 4200
-F 0 "D?" V 5296 4288 50  0000 L CNN
+F 0 "D5" V 5296 4288 50  0000 L CNN
 F 1 "BAT54S" V 5205 4288 50  0000 L CNN
 F 2 "Package_TO_SOT_SMD:SOT-23" H 5325 4325 50  0001 L CNN
@@
 Connection ~ 6350 2850
 $Comp
-L Diode:1N4148 D?
+L Diode:1N4148 D6
 U 1 1 5E95B772
 P 6550 3250
-F 0 "D?" V 6504 3329 50  0000 L CNN
+F 0 "D6" V 6504 3329 50  0000 L CNN
 F 1 "SMAJ13CA" V 6595 3329 50  0000 L CNN
 F 2 "Diode_THT:D_DO-35_SOD27_P7.62mm_Horizontal" H 6550 3075 50  0001 C CNN
@@
 Wire Wire Line
 	6900 2850 6900 3200
-Wire Wire Line
-	6900 3200 7900 3200
 Connection ~ 6550 2850
-Text Label 7600 3200 0    50   ~ 0
-CP
-$Comp
-L Diode:BAT54S D?
+Text Label 7500 3200 0    50   ~ 0
+CP_con
+$Comp
+L Diode:BAT54S D7
 U 1 1 5E9604E7
 P 7100 2800
-F 0 "D?" V 7146 2888 50  0000 L CNN
+F 0 "D7" V 7146 2888 50  0000 L CNN
 F 1 "BAT54S" V 7055 2888 50  0000 L CNN
 F 2 "Package_TO_SOT_SMD:SOT-23" H 7175 2925 50  0001 L CNN
@@
 	7300 2700 7450 2700
 $Comp
-L Device:R_Small R?
+L Device:R_Small R24
 U 1 1 5E968C58
 P 7550 2700
-F 0 "R?" V 7354 2700 50  0000 C CNN
+F 0 "R24" V 7354 2700 50  0000 C CNN
 F 1 "100" V 7445 2700 50  0000 C CNN
 F 2 "" H 7550 2700 50  0001 C CNN
@@
 Text HLabel 7900 3100 0    50   Input ~ 0
 Lock_W
-Wire Notes Line
-	7150 3150 7150 3750
-Wire Notes Line
-	7150 3750 7500 3750
-Wire Notes Line
-	7500 3750 7500 3150
-Wire Notes Line
-	7500 3150 7150 3150
-Text Notes 7100 3450 0    50   ~ 0
-Reed Relays!
 Text HLabel 3850 3650 0    50   Output ~ 0
 PP
@@
 Text HLabel 7300 2600 1    50   Output ~ 0
 Button
-Text HLabel 3850 5000 0    50   Input ~ 0
+Text HLabel 3600 5550 0    50   Input ~ 0
 Reed_Relay
 Wire Wire Line
-	3850 5000 4250 5000
+	3600 5550 4000 5550
 Wire Notes Line
 	5050 800  5050 2450
@@
 Text Notes 5400 3250 2    50   ~ 0
 Comparator\n
+$Comp
+L smartevse:Reed_Relay_DPST_NC K1
+U 1 1 5E9A6E64
+P 5950 5550
+F 0 "K1" V 5283 5550 50  0000 C CNN
+F 1 "Reed Relay DPST NC" V 5374 5550 50  0000 C CNN
+F 2 "Relay_THT:Relay_StandexMeder_DIP_LowProfile" H 6450 5500 50  0001 L CNN
+F 3 "https://standexelectronics.com/wp-content/uploads/datasheet_reed_relay_DIP.pdf" H 5950 5550 50  0001 C CNN
+	1    5950 5550
+	0    1    1    0
+$EndComp
+Wire Wire Line
+	5600 3650 7150 3650
+Connection ~ 5600 3650
+Wire Wire Line
+	6900 3200 7150 3200
+Wire Wire Line
+	7500 3650 7800 3650
+Wire Wire Line
+	7900 3200 7500 3200
+Text Label 6950 3200 0    50   ~ 0
+CP_to_relay
+Text Label 6950 3650 0    50   ~ 0
+PP_to_relay
+Wire Notes Line width 20 style solid
+	7400 3150 7400 3650
+Wire Notes Line
+	7400 3650 7450 3650
+Wire Notes Line width 20 style solid rgb(70, 194, 85)
+	7450 3650 7450 3150
+Wire Notes Line
+	7450 3150 7400 3150
+Text Label 5500 5950 2    50   ~ 0
+PP_to_relay
+Text Label 5500 5650 2    50   ~ 0
+CP_to_relay
+Wire Wire Line
+	5500 5650 5650 5650
+Wire Wire Line
+	5500 5950 5650 5950
+Wire Wire Line
+	6250 5650 6400 5650
+Wire Wire Line
+	6400 5950 6250 5950
+Text Label 6400 5650 0    50   ~ 0
+CP_con
+Text Label 6400 5950 0    50   ~ 0
+PP_con
+Wire Wire Line
+	5650 5250 4850 5250
+Wire Wire Line
+	4850 5250 4850 5350
+Wire Wire Line
+	6250 5250 6500 5250
+Wire Wire Line
+	6500 5250 6500 5000
+$Comp
+L power:+12V #PWR029
+U 1 1 5E9D6AB9
+P 6500 5000
+F 0 "#PWR029" H 6500 4850 50  0001 C CNN
+F 1 "+12V" H 6515 5173 50  0000 C CNN
+F 2 "" H 6500 5000 50  0001 C CNN
+F 3 "" H 6500 5000 50  0001 C CNN
+	1    6500 5000
+	1    0    0    -1
+$EndComp
+$Comp
+L Transistor_BJT:2N3904 Q2
+U 1 1 5E9D7037
+P 4750 5550
+F 0 "Q2" H 4941 5596 50  0000 L CNN
+F 1 "Drive Transistor" H 4650 5350 50  0000 L CNN
+F 2 "Package_TO_SOT_THT:TO-92_Inline" H 4950 5475 50  0001 L CIN
+F 3 "https://www.fairchildsemi.com/datasheets/2N/2N3904.pdf" H 4750 5550 50  0001 L CNN
+	1    4750 5550
+	1    0    0    -1
+$EndComp
+$Comp
+L Device:R_Small R14
+U 1 1 5E9D987E
+P 4100 5550
+F 0 "R14" V 3904 5550 50  0000 C CNN
+F 1 "2.2k" V 3995 5550 50  0000 C CNN
+F 2 "" H 4100 5550 50  0001 C CNN
+F 3 "~" H 4100 5550 50  0001 C CNN
+	1    4100 5550
+	0    1    1    0
+$EndComp
+$Comp
+L Device:R_Small R17
+U 1 1 5E9DA4DD
+P 4350 5800
+F 0 "R17" H 4291 5754 50  0000 R CNN
+F 1 "22k" H 4291 5845 50  0000 R CNN
+F 2 "" H 4350 5800 50  0001 C CNN
+F 3 "~" H 4350 5800 50  0001 C CNN
+	1    4350 5800
+	-1   0    0    1
+$EndComp
+Wire Wire Line
+	4850 5750 4850 6000
+Wire Wire Line
+	4850 6000 4600 6000
+Wire Wire Line
+	4350 6000 4350 5900
+Wire Wire Line
+	4350 5700 4350 5550
+Wire Wire Line
+	4350 5550 4200 5550
+Wire Wire Line
+	4350 5550 4550 5550
+Connection ~ 4350 5550
+$Comp
+L power:GND #PWR028
+U 1 1 5E9E16AA
+P 4600 6000
+F 0 "#PWR028" H 4600 5750 50  0001 C CNN
+F 1 "GND" H 4605 5827 50  0000 C CNN
+F 2 "" H 4600 6000 50  0001 C CNN
+F 3 "" H 4600 6000 50  0001 C CNN
+	1    4600 6000
+	1    0    0    -1
+$EndComp
+Connection ~ 4600 6000
+Wire Wire Line
+	4600 6000 4350 6000
 $EndSCHEMATC

Commit message: Update schematic with suggestions
Changed lines of the file:
@@
 U 1 1 5E968C58
 P 7550 2700
-F 0 "R24" V 7354 2700 50  0000 C CNN
+F 0 "R24" V 7650 2700 50  0000 C CNN
 F 1 "100" V 7445 2700 50  0000 C CNN
 F 2 "" H 7550 2700 50  0001 C CNN

Commit message: Edit schematic
Moved CT input to J2
Parts:
- added C? (x3): 100n, symbol Device:C_Small
- added R? (x3): 100, symbol Device:R_Small
- added R? (x3): 22, symbol Device:R_Small
- added R? (x2): 10k, symbol Device:R_Small
- J2: symbol Connector:Screw_Terminal_01x12 -> Connector:Screw_Terminal_01x20
Connections:
- net labels added: BIAS, CT0, CT0_K, CT0_L, CT1, CT1_K, CT1_L, CT2, CT2_K, CT2_L
- wire segments 88 -> 126
Other:
- note added: "Current Transformer Input Section\n"
- note added: "VDD/2 Bias Voltage for CT input\n"
- moved on the sheet: F1, K1, Q2, R14, R17, R24

Commit message: Edit schematic to rev0.6
Updated schematic with ESP32, CT inputs moved, Button input circuit new.
Temp sens removed, will use internal sensor in ATmega4808
Parts:
- added D?: 3.3V Zener, symbol Device:D_Zener_Small
- added D?: Only needed if not included in relay, symbol Device:D_Small
- added R?: 33, symbol Device:R_Small
- Q2: value Drive Transistor -> 2N2222 or similar; footprint Package_TO_SOT_THT:TO-92_Inline -> (none)
- gave numbers to parts that had none: 11
Connections:
- net +12V: now also F1.1, D?.1 (K)
- net Button: now also D?.1 (K), R?.1
- net GND: now also D?.2 (A), R?.2
- net 12V_Fused: now reaches F1.2, J2.3 (Pin_3)
- net at K1.2, Q2.3 (C): now also D?.2 (A)
- no-connect marks 1 -> 3
Changed lines of the file:
@@
 Sheet 4 4
 Title ""
-Date "2020-05-14"
-Rev "0.5"
+Date "2020-05-18"
+Rev "0.6"
 Comp ""
 Comment1 "DONE: CT inputs on J2"
 Comment2 "TODO: Det. Q2, R14, R17, verify relay circuit"
-Comment3 ""
-Comment4 ""
+Comment3 "TODO: verify CT bias voltage divider & CT circuit"
+Comment4 "DONE: voltage divider & zener diode on button input"
 $EndDescr
 $Comp
@@
 $EndComp
 Connection ~ 6200 1150
-Wire Wire Line
-	6200 1150 7800 1150
 $Comp
 L Device:Opamp_Dual_Generic U11
@@
 	1    0    0    -1
 $EndComp
-Wire Wire Line
-	7900 2800 7900 2700
-Wire Wire Line
-	7900 2700 8050 2700
 $Comp
 L Device:R_Small R24
@@
 Text HLabel 3850 3650 0    50   Output ~ 0
 PP
-Wire Wire Line
-	7900 2600 7900 2700
-Connection ~ 7900 2700
-Text HLabel 7900 2600 1    50   Output ~ 0
+Text HLabel 7500 2300 1    50   Output ~ 0
 Button
 Text HLabel 6000 5400 0    50   Input ~ 0
@@
 PP_con
 Wire Wire Line
-	7850 5100 7050 5100
+	7850 5100 7550 5100
 Wire Wire Line
 	7050 5100 7050 5200
 Wire Wire Line
-	8450 5100 8700 5100
+	8450 5100 8500 5100
 Wire Wire Line
 	8700 5100 8700 4850
@@
 P 6950 5400
 F 0 "Q2" H 7141 5446 50  0000 L CNN
-F 1 "Drive Transistor" H 6850 5200 50  0000 L CNN
-F 2 "Package_TO_SOT_THT:TO-92_Inline" H 7150 5325 50  0001 L CIN
+F 1 "2N2222 or similar" H 6850 5200 50  0000 L CNN
+F 2 "" H 7150 5325 50  0001 L CIN
 F 3 "https://www.fairchildsemi.com/datasheets/2N/2N3904.pdf" H 6950 5400 50  0001 L CNN
 	1    6950 5400
@@
 P 1300 5450
 AR Path="/5E98FA8A/5EC179B9" Ref="#PWR?"  Part="1"
-AR Path="/5E903BF9/5EC179B9" Ref="#PWR?"  Part="1"
-F 0 "#PWR?" H 1300 5200 50  0001 C CNN
+AR Path="/5E903BF9/5EC179B9" Ref="#PWR039"  Part="1"
+F 0 "#PWR039" H 1300 5200 50  0001 C CNN
 F 1 "GND" H 1305 5277 50  0000 C CNN
 F 2 "" H 1300 5450 50  0001 C CNN
@@
 P 1300 5350
 AR Path="/5E98FA8A/5EC179C0" Ref="C?"  Part="1"
-AR Path="/5E903BF9/5EC179C0" Ref="C?"  Part="1"
-F 0 "C?" H 1392 5396 50  0000 L CNN
+AR Path="/5E903BF9/5EC179C0" Ref="C23"  Part="1"
+F 0 "C23" H 1392 5396 50  0000 L CNN
 F 1 "100n" H 1392 5305 50  0000 L CNN
 F 2 "" H 1300 5350 50  0001 C CNN
@@
 P 1650 5200
 AR Path="/5E98FA8A/5EC179D4" Ref="R?"  Part="1"
-AR Path="/5E903BF9/5EC179D4" Ref="R?"  Part="1"
-F 0 "R?" V 1454 5200 50  0000 C CNN
+AR Path="/5E903BF9/5EC179D4" Ref="R28"  Part="1"
+F 0 "R28" V 1454 5200 50  0000 C CNN
 F 1 "100" V 1545 5200 50  0000 C CNN
 F 2 "" H 1650 5200 50  0001 C CNN
@@
 P 1950 5450
 AR Path="/5E98FA8A/5EC179DA" Ref="R?"  Part="1"
-AR Path="/5E903BF9/5EC179DA" Ref="R?"  Part="1"
-F 0 "R?" H 2009 5496 50  0000 L CNN
+AR Path="/5E903BF9/5EC179DA" Ref="R31"  Part="1"
+F 0 "R31" H 2009 5496 50  0000 L CNN
 F 1 "22" H 2009 5405 50  0000 L CNN
 F 2 "" H 1950 5450 50  0001 C CNN
@@
 P 1300 6350
 AR Path="/5E98FA8A/5EC179E9" Ref="#PWR?"  Part="1"
-AR Path="/5E903BF9/5EC179E9" Ref="#PWR?"  Part="1"
-F 0 "#PWR?" H 1300 6100 50  0001 C CNN
+AR Path="/5E903BF9/5EC179E9" Ref="#PWR040"  Part="1"
+F 0 "#PWR040" H 1300 6100 50  0001 C CNN
 F 1 "GND" H 1305 6177 50  0000 C CNN
 F 2 "" H 1300 6350 50  0001 C CNN
@@
 P 1300 6250
 AR Path="/5E98FA8A/5EC179F0" Ref="C?"  Part="1"
-AR Path="/5E903BF9/5EC179F0" Ref="C?"  Part="1"
-F 0 "C?" H 1392 6296 50  0000 L CNN
+AR Path="/5E903BF9/5EC179F0" Ref="C24"  Part="1"
+F 0 "C24" H 1392 6296 50  0000 L CNN
 F 1 "100n" H 1392 6205 50  0000 L CNN
 F 2 "" H 1300 6250 50  0001 C CNN
@@
 P 1650 6100
 AR Path="/5E98FA8A/5EC17A04" Ref="R?"  Part="1"
-AR Path="/5E903BF9/5EC17A04" Ref="R?"  Part="1"
-F 0 "R?" V 1454 6100 50  0000 C CNN
+AR Path="/5E903BF9/5EC17A04" Ref="R29"  Part="1"
+F 0 "R29" V 1454 6100 50  0000 C CNN
 F 1 "100" V 1545 6100 50  0000 C CNN
 F 2 "" H 1650 6100 50  0001 C CNN
@@
 P 1950 6350
 AR Path="/5E98FA8A/5EC17A0A" Ref="R?"  Part="1"
-AR Path="/5E903BF9/5EC17A0A" Ref="R?"  Part="1"
-F 0 "R?" H 2009 6396 50  0000 L CNN
+AR Path="/5E903BF9/5EC17A0A" Ref="R32"  Part="1"
+F 0 "R32" H 2009 6396 50  0000 L CNN
 F 1 "22" H 2009 6305 50  0000 L CNN
 F 2 "" H 1950 6350 50  0001 C CNN
@@
 P 1300 7250
 AR Path="/5E98FA8A/5EC17A19" Ref="#PWR?"  Part="1"
-AR Path="/5E903BF9/5EC17A19" Ref="#PWR?"  Part="1"
-F 0 "#PWR?" H 1300 7000 50  0001 C CNN
+AR Path="/5E903BF9/5EC17A19" Ref="#PWR041"  Part="1"
+F 0 "#PWR041" H 1300 7000 50  0001 C CNN
 F 1 "GND" H 1305 7077 50  0000 C CNN
 F 2 "" H 1300 7250 50  0001 C CNN
@@
 P 1300 7150
 AR Path="/5E98FA8A/5EC17A20" Ref="C?"  Part="1"
-AR Path="/5E903BF9/5EC17A20" Ref="C?"  Part="1"
-F 0 "C?" H 1392 7196 50  0000 L CNN
+AR Path="/5E903BF9/5EC17A20" Ref="C25"  Part="1"
+F 0 "C25" H 1392 7196 50  0000 L CNN
 F 1 "100n" H 1392 7105 50  0000 L CNN
 F 2 "" H 1300 7150 50  0001 C CNN
@@
 P 1650 7000
 AR Path="/5E98FA8A/5EC17A34" Ref="R?"  Part="1"
-AR Path="/5E903BF9/5EC17A34" Ref="R?"  Part="1"
-F 0 "R?" V 1454 7000 50  0000 C CNN
+AR Path="/5E903BF9/5EC17A34" Ref="R30"  Part="1"
+F 0 "R30" V 1454 7000 50  0000 C CNN
 F 1 "100" V 1545 7000 50  0000 C CNN
 F 2 "" H 1650 7000 50  0001 C CNN
@@
 P 1950 7250
 AR Path="/5E98FA8A/5EC17A3A" Ref="R?"  Part="1"
-AR Path="/5E903BF9/5EC17A3A" Ref="R?"  Part="1"
-F 0 "R?" H 2009 7296 50  0000 L CNN
+AR Path="/5E903BF9/5EC17A3A" Ref="R33"  Part="1"
+F 0 "R33" H 2009 7296 50  0000 L CNN
 F 1 "22" H 2009 7205 50  0000 L CNN
 F 2 "" H 1950 7250 50  0001 C CNN
@@
 CT2_K
 $Comp
-L power:+3.3V #PWR?
+L power:+3.3V #PWR042
 U 1 1 5EC624C4
 P 1500 3550
-F 0 "#PWR?" H 1500 3400 50  0001 C CNN
+F 0 "#PWR042" H 1500 3400 50  0001 C CNN
 F 1 "+3.3V" H 1515 3723 50  0000 C CNN
 F 2 "" H 1500 3550 50  0001 C CNN
@@
 $EndComp
 $Comp
-L power:GND #PWR?
+L power:GND #PWR043
 U 1 1 5EC624CA
 P 1500 4250
-F 0 "#PWR?" H 1500 4000 50  0001 C CNN
+F 0 "#PWR043" H 1500 4000 50  0001 C CNN
 F 1 "GND" H 1505 4077 50  0000 C CNN
 F 2 "" H 1500 4250 50  0001 C CNN
@@
 $EndComp
 $Comp
-L Device:R_Small R?
+L Device:R_Small R27
 U 1 1 5EC624D0
 P 1500 4050
-F 0 "R?" H 1559 4096 50  0000 L CNN
+F 0 "R27" H 1559 4096 50  0000 L CNN
 F 1 "10k" H 1559 4005 50  0000 L CNN
 F 2 "" H 1500 4050 50  0001 C CNN
@@
 $EndComp
 $Comp
-L Device:R_Small R?
+L Device:R_Small R26
 U 1 1 5EC624D6
 P 1500 3700
-F 0 "R?" H 1559 3746 50  0000 L CNN
+F 0 "R26" H 1559 3746 50  0000 L CNN
 F 1 "10k" H 1559 3655 50  0000 L CNN
 F 2 "" H 1500 3700 50  0001 C CNN
@@
 Text Notes 850  4750 0    50   ~ 0
 VDD/2 Bias Voltage for CT input\n
-Wire Wire Line
-	7300 2800 7900 2800
+NoConn ~ 8500 3400
+NoConn ~ 8500 3500
+Wire Wire Line
+	6200 1150 8400 1150
+$Comp
+L Device:R_Small R?
+U 1 1 5ECD3565
+P 7500 2800
+F 0 "R?" H 7550 2850 50  0000 L CNN
+F 1 "33" H 7559 2755 50  0000 L CNN
+F 2 "" H 7500 2800 50  0001 C CNN
+F 3 "~" H 7500 2800 50  0001 C CNN
+	1    7500 2800
+	1    0    0    -1
+$EndComp
+Wire Wire Line
+	7500 2700 7700 2700
+Wire Wire Line
+	7500 2700 7500 2300
+Connection ~ 7500 2700
+Wire Wire Line
+	7300 2800 7300 2700
+Wire Wire Line
+	7300 2700 7500 2700
+$Comp
+L Device:D_Zener_Small D?
+U 1 1 5ECE49DD
+P 7700 2800
+F 0 "D?" V 7654 2868 50  0000 L CNN
+F 1 "3.3V Zener" V 7745 2868 50  0000 L CNN
+F 2 "" V 7700 2800 50  0001 C CNN
+F 3 "~" V 7700 2800 50  0001 C CNN
+	1    7700 2800
+	0    1    1    0
+$EndComp
+Connection ~ 7100 3100
+Wire Wire Line
+	7500 2900 7500 3100
+Wire Wire Line
+	7100 3100 7500 3100
+Connection ~ 7500 2900
+Connection ~ 7700 2700
+Wire Wire Line
+	7700 2900 7500 2900
+Wire Wire Line
+	7700 2700 8050 2700
+Text Label 8400 2400 2    50   ~ 0
+12V_Fused
+$Comp
+L Device:D_Small D?
+U 1 1 5ECFD670
+P 8100 4600
+F 0 "D?" H 8100 4395 50  0000 C CNN
+F 1 "Only needed if not included in relay" H 8100 4486 50  0000 C CNN
+F 2 "" V 8100 4600 50  0001 C CNN
+F 3 "~" V 8100 4600 50  0001 C CNN
+	1    8100 4600
+	-1   0    0    1
+$EndComp
+Wire Wire Line
+	8200 4600 8500 4600
+Wire Wire Line
+	8500 4600 8500 5100
+Connection ~ 8500 5100
+Wire Wire Line
+	8500 5100 8700 5100
+Wire Wire Line
+	8000 4600 7550 4600
+Wire Wire Line
+	7550 4600 7550 5100
+Connection ~ 7550 5100
+Wire Wire Line
+	7550 5100 7050 5100
 $EndSCHEMATC
