File: circuit/analog_section_low_voltage.sch (KiCad schematic (older format))
At the start: 36 parts, among them J2 Screw_Terminal_01x18, U11 LM7332, U12 CPC1114N, U13 CPC1114N

Commit message: Update first layout draft
Parts:
- R13: footprint Resistor_SMD:R_0805_2012Metric_Pad1.15x1.40mm_HandSolder -> Resistor_SMD:R_0603_1608Metric_Pad1.05x0.95mm_HandSolder
Changed lines of the file:
@@
 F 0 "R13" H 4009 2296 50  0000 L CNN
 F 1 "40.2k" H 4009 2205 50  0000 L CNN
-F 2 "Resistor_SMD:R_0805_2012Metric_Pad1.15x1.40mm_HandSolder" H 3950 2250 50  0001 C CNN
+F 2 "Resistor_SMD:R_0603_1608Metric_Pad1.05x0.95mm_HandSolder" H 3950 2250 50  0001 C CNN
 F 3 "~" H 3950 2250 50  0001 C CNN
 F 4 "" H 3950 2250 50  0001 C CNN "Part"

Commit message: Update doc
Parts:
- removed D8: 3.3V Zener, Diode_SMD:D_SOD-323_HandSoldering, symbol Device:D_Zener_Small
- removed J2: Screw_Terminal_01x18, atmevse-footprints:CUI_TB004-508-18BE, symbol Connector:Screw_Terminal_01x18
- removed R34: 33, Resistor_SMD:R_0603_1608Metric_Pad1.05x0.95mm_HandSolder, symbol Device:R_Small
- added D? (x4): BAT54S, Package_TO_SOT_SMD:SOT-23, symbol Diode:BAT54S
- added J? (x2): Screw_Terminal_01x09, symbol Connector:Screw_Terminal_01x09
- R24: value 100 -> 1k
Connections:
- net +3V3: now also D?.2, D?.2, D?.2, D?.2
- net 12V_Fused: now also J?.6 (Pin_6)
- net BIAS: now also J?.5 (Pin_5), J?.7 (Pin_7), J?.9 (Pin_9)
- net CP: now also D?.3
- net CP_con: now also J?.1 (Pin_1)
- net CT0: now also D?.3
- net CT0_L: now also J?.4 (Pin_4)
- net CT1: now also D?.3
- net CT1_L: now also J?.6 (Pin_6)
- net CT2: now also D?.3
- net CT2_L: now also J?.8 (Pin_8)
- net GND: now also D?.1, D?.1, D?.1, D?.1, J?.3 (Pin_3)
- net LED: now also J?.4 (Pin_4)
- net Lock_B: now also J?.7 (Pin_7)
- net Lock_R: now also J?.8 (Pin_8)
- net Lock_W: now also J?.9 (Pin_9)
- net PP_con: now also J?.2 (Pin_2)
- net RS485_A: now also J?.1 (Pin_1)
- net RS485_B: now also J?.2 (Pin_2)
- net at R24.1: now also J?.5 (Pin_5)
Other:
- moved on the sheet: C23, C24, C25, D7, F1, R24, R28, R29, R30, R31, R32, R33

Commit message: Testing build
Parts:
- gave numbers to parts that had none: 6
Changed lines of the file:
@@
 $Descr A4 11693 8268
 encoding utf-8
-Sheet 4 5
+Sheet 4 4
 Title "FGCCS-Ctrl22"
 Date "2020-08-11"
@@
 $EndComp
 $Comp
-L Connector:Screw_Terminal_01x09 J?
+L Connector:Screw_Terminal_01x09 J6
 U 1 1 5F3444D0
 P 8700 2600
-F 0 "J?" H 8780 2642 50  0000 L CNN
+F 0 "J6" H 8780 2642 50  0000 L CNN
 F 1 "Screw_Terminal_01x09" H 8780 2551 50  0000 L CNN
 F 2 "" H 8700 2600 50  0001 C CNN
@@
 $EndComp
 $Comp
-L Connector:Screw_Terminal_01x09 J?
+L Connector:Screw_Terminal_01x09 J7
 U 1 1 5F34567E
 P 8700 3500
-F 0 "J?" H 8780 3542 50  0000 L CNN
+F 0 "J7" H 8780 3542 50  0000 L CNN
 F 1 "Screw_Terminal_01x09" H 8780 3451 50  0000 L CNN
 F 2 "" H 8700 3500 50  0001 C CNN
@@
 NoConn ~ 8500 3300
 $Comp
-L Diode:BAT54S D?
+L Diode:BAT54S D8
 U 1 1 5F402191
 P 1350 5500
-F 0 "D?" V 1396 5588 50  0000 L CNN
+F 0 "D8" V 1396 5588 50  0000 L CNN
 F 1 "BAT54S" V 1305 5588 50  0000 L CNN
 F 2 "Package_TO_SOT_SMD:SOT-23" H 1425 5625 50  0001 L CNN
@@
 $EndComp
 $Comp
-L Diode:BAT54S D?
+L Diode:BAT54S D9
 U 1 1 5F403CE8
 P 1350 6400
-F 0 "D?" V 1396 6488 50  0000 L CNN
+F 0 "D9" V 1396 6488 50  0000 L CNN
 F 1 "BAT54S" V 1305 6488 50  0000 L CNN
 F 2 "Package_TO_SOT_SMD:SOT-23" H 1425 6525 50  0001 L CNN
@@
 $EndComp
 $Comp
-L Diode:BAT54S D?
+L Diode:BAT54S D10
 U 1 1 5F404582
 P 1350 7300
-F 0 "D?" V 1396 7388 50  0000 L CNN
+F 0 "D10" V 1396 7388 50  0000 L CNN
 F 1 "BAT54S" V 1305 7388 50  0000 L CNN
 F 2 "Package_TO_SOT_SMD:SOT-23" H 1425 7425 50  0001 L CNN
@@
 $EndComp
 $Comp
-L power:GND #PWR?
+L power:GND #PWR045
 U 1 1 5F405023
 P 1350 5800
-F 0 "#PWR?" H 1350 5550 50  0001 C CNN
+F 0 "#PWR045" H 1350 5550 50  0001 C CNN
 F 1 "GND" H 1355 5627 50  0000 C CNN
 F 2 "" H 1350 5800 50  0001 C CNN
@@
 $EndComp
 $Comp
-L power:GND #PWR?
+L power:GND #PWR046
 U 1 1 5F405A5C
 P 1350 6700
-F 0 "#PWR?" H 1350 6450 50  0001 C CNN
+F 0 "#PWR046" H 1350 6450 50  0001 C CNN
 F 1 "GND" H 1355 6527 50  0000 C CNN
 F 2 "" H 1350 6700 50  0001 C CNN
@@
 $EndComp
 $Comp
-L power:GND #PWR?
+L power:GND #PWR047
 U 1 1 5F405D93
 P 1350 7600
-F 0 "#PWR?" H 1350 7350 50  0001 C CNN
+F 0 "#PWR047" H 1350 7350 50  0001 C CNN
 F 1 "GND" H 1355 7427 50  0000 C CNN
 F 2 "" H 1350 7600 50  0001 C CNN
@@
 	1350 5200 1350 5050
 $Comp
-L power:+3.3V #PWR?
+L power:+3.3V #PWR044
 U 1 1 5F435027
 P 1350 5050
-F 0 "#PWR?" H 1350 4900 50  0001 C CNN
+F 0 "#PWR044" H 1350 4900 50  0001 C CNN
 F 1 "+3.3V" H 1365 5223 50  0000 C CNN
 F 2 "" H 1350 5050 50  0001 C CNN
@@
 $EndComp
 $Comp
-L power:+3.3V #PWR?
+L power:+3.3V #PWR048
 U 1 1 5F43561C
 P 1500 5850
-F 0 "#PWR?" H 1500 5700 50  0001 C CNN
+F 0 "#PWR048" H 1500 5700 50  0001 C CNN
 F 1 "+3.3V" H 1515 6023 50  0000 C CNN
 F 2 "" H 1500 5850 50  0001 C CNN
@@
 	1500 5850 1500 6100
 $Comp
-L power:+3.3V #PWR?
+L power:+3.3V #PWR049
 U 1 1 5F435A9E
 P 1500 6750
-F 0 "#PWR?" H 1500 6600 50  0001 C CNN
+F 0 "#PWR049" H 1500 6600 50  0001 C CNN
 F 1 "+3.3V" H 1515 6923 50  0000 C CNN
 F 2 "" H 1500 6750 50  0001 C CNN
@@
 $EndComp
 $Comp
-L Diode:BAT54S D?
+L Diode:BAT54S D11
 U 1 1 5F4367A4
 P 3450 2000
-F 0 "D?" V 3496 2088 50  0000 L CNN
+F 0 "D11" V 3496 2088 50  0000 L CNN
 F 1 "BAT54S" V 3405 2088 50  0000 L CNN
 F 2 "Package_TO_SOT_SMD:SOT-23" H 3525 2125 50  0001 L CNN
@@
 $EndComp
 $Comp
-L power:+3.3V #PWR?
+L power:+3.3V #PWR050
 U 1 1 5F43902A
 P 3450 1700
-F 0 "#PWR?" H 3450 1550 50  0001 C CNN
+F 0 "#PWR050" H 3450 1550 50  0001 C CNN
 F 1 "+3.3V" H 3465 1873 50  0000 C CNN
 F 2 "" H 3450 1700 50  0001 C CNN
@@
 $EndComp
 $Comp
-L power:GND #PWR?
+L power:GND #PWR051
 U 1 1 5F439C89
 P 3450 2300
-F 0 "#PWR?" H 3450 2050 50  0001 C CNN
+F 0 "#PWR051" H 3450 2050 50  0001 C CNN
 F 1 "GND" H 3455 2127 50  0000 C CNN
 F 2 "" H 3450 2300 50  0001 C CNN

Commit message: Finish Revision 1.1 layout
Parts:
- D10, D11, D8, D9: footprint Package_TO_SOT_SMD:SOT-23 -> Package_TO_SOT_SMD:SOT-23_Handsoldering
- J6: footprint (none) -> atmevse-footprints:lv_screw_9pin_1
- J7: footprint (none) -> atmevse-footprints:lv_screw_9pin_2
Changed lines of the file:
@@
 F 0 "J6" H 8780 2642 50  0000 L CNN
 F 1 "Screw_Terminal_01x09" H 8780 2551 50  0000 L CNN
-F 2 "" H 8700 2600 50  0001 C CNN
+F 2 "atmevse-footprints:lv_screw_9pin_1" H 8700 2600 50  0001 C CNN
 F 3 "~" H 8700 2600 50  0001 C CNN
 	1    8700 2600
@@
 F 0 "J7" H 8780 3542 50  0000 L CNN
 F 1 "Screw_Terminal_01x09" H 8780 3451 50  0000 L CNN
-F 2 "" H 8700 3500 50  0001 C CNN
+F 2 "atmevse-footprints:lv_screw_9pin_2" H 8700 3500 50  0001 C CNN
 F 3 "~" H 8700 3500 50  0001 C CNN
 	1    8700 3500
@@
 F 0 "D8" V 1396 5588 50  0000 L CNN
 F 1 "BAT54S" V 1305 5588 50  0000 L CNN
-F 2 "Package_TO_SOT_SMD:SOT-23" H 1425 5625 50  0001 L CNN
+F 2 "Package_TO_SOT_SMD:SOT-23_Handsoldering" H 1425 5625 50  0001 L CNN
 F 3 "https://www.diodes.com/assets/Datasheets/ds11005.pdf" H 1230 5500 50  0001 C CNN
 	1    1350 5500
@@
 F 0 "D9" V 1396 6488 50  0000 L CNN
 F 1 "BAT54S" V 1305 6488 50  0000 L CNN
-F 2 "Package_TO_SOT_SMD:SOT-23" H 1425 6525 50  0001 L CNN
+F 2 "Package_TO_SOT_SMD:SOT-23_Handsoldering" H 1425 6525 50  0001 L CNN
 F 3 "https://www.diodes.com/assets/Datasheets/ds11005.pdf" H 1230 6400 50  0001 C CNN
 	1    1350 6400
@@
 F 0 "D10" V 1396 7388 50  0000 L CNN
 F 1 "BAT54S" V 1305 7388 50  0000 L CNN
-F 2 "Package_TO_SOT_SMD:SOT-23" H 1425 7425 50  0001 L CNN
+F 2 "Package_TO_SOT_SMD:SOT-23_Handsoldering" H 1425 7425 50  0001 L CNN
 F 3 "https://www.diodes.com/assets/Datasheets/ds11005.pdf" H 1230 7300 50  0001 C CNN
 	1    1350 7300
@@
 F 0 "D11" V 3496 2088 50  0000 L CNN
 F 1 "BAT54S" V 3405 2088 50  0000 L CNN
-F 2 "Package_TO_SOT_SMD:SOT-23" H 3525 2125 50  0001 L CNN
+F 2 "Package_TO_SOT_SMD:SOT-23_Handsoldering" H 3525 2125 50  0001 L CNN
 F 3 "https://www.diodes.com/assets/Datasheets/ds11005.pdf" H 3330 2000 50  0001 C CNN
 	1    3450 2000
