File: circuit/atmega4808_and_peripherals.sch (KiCad schematic (older format))
At the start: 30 parts, among them J3 Conn_01x04, J4 Conn_02x04_Top_Bottom, J5 Conn_02x04_Top_Bottom, Q1 BSS138, U10 ATmega4808-X, U7 SN65HVD72C, U8 FAN3214TMX, U9 ESP32-WROOM-32

Commit message: Finish schematic rev1 and footprint assignment
Parts:
- C12: PartNo (none) -> 871-B41231A4109M000
- C13, C14, C15, C17: footprint Capacitor_SMD:C_0603_1608Metric_Pad1.05x0.95mm_HandSolder -> Capacitor_SMD:C_0805_2012Metric_Pad1.15x1.40mm_HandSolder; PartNo (none) -> 963-EMF212B7104KGHT
- C16: footprint Capacitor_Tantalum_SMD:CP_EIA-7343-15_Kemet-W_Pad2.25x2.55mm_HandSolder -> Capacitor_SMD:C_0805_2012Metric_Pad1.15x1.40mm_HandSolder; PartNo (none) -> 581-TLCR107M006RTA
- C21: footprint Capacitor_SMD:C_0603_1608Metric_Pad1.05x0.95mm_HandSolder -> Capacitor_SMD:C_0805_2012Metric_Pad1.15x1.40mm_HandSolder; PartNo (none) -> 77-VJ0805A102KXAAC
- C22: footprint Capacitor_SMD:C_0603_1608Metric_Pad1.05x0.95mm_HandSolder -> Capacitor_SMD:C_0805_2012Metric_Pad1.15x1.40mm_HandSolder; PartNo (none) -> 77-VJ805Y105KXARW1BC
- J3: PartNo 710-61304011121 -> 710-61304011121
- J4, J5: PartNo 710-61300821121 -> 710-61300821121
- U7: PartNo (none) -> 595-SN65HVD72D
- U8: PartNo (none) -> 512-FAN3214TMX
Changed lines of the file:
@@
 Sheet 3 4
 Title ""
-Date "2020-05-29"
-Rev "0.7"
+Date "2020-06-01"
+Rev "1.0"
 Comp ""
 Comment1 "DONE: ESP32 circuit"
@@
 F 0 "C17" H 7392 4046 50  0000 L CNN
 F 1 "100n" H 7392 3955 50  0000 L CNN
-F 2 "Capacitor_SMD:C_0603_1608Metric_Pad1.05x0.95mm_HandSolder" H 7300 4000 50  0001 C CNN
+F 2 "Capacitor_SMD:C_0805_2012Metric_Pad1.15x1.40mm_HandSolder" H 7300 4000 50  0001 C CNN
 F 3 "~" H 7300 4000 50  0001 C CNN
 F 4 "" H 7300 4000 50  0001 C CNN "Part"
-F 5 "" H 7300 4000 50  0001 C CNN "PartNo"
+F 5 "963-EMF212B7104KGHT " H 7300 4000 50  0001 C CNN "PartNo"
 F 6 "Mouser" H 7300 4000 50  0001 C CNN "Supplier"
 	1    7300 4000
@@
 F 0 "C15" V 5521 5000 50  0000 C CNN
 F 1 "100n" V 5612 5000 50  0000 C CNN
-F 2 "Capacitor_SMD:C_0603_1608Metric_Pad1.05x0.95mm_HandSolder" H 5750 5000 50  0001 C CNN
+F 2 "Capacitor_SMD:C_0805_2012Metric_Pad1.15x1.40mm_HandSolder" H 5750 5000 50  0001 C CNN
 F 3 "~" H 5750 5000 50  0001 C CNN
 F 4 "" H 5750 5000 50  0001 C CNN "Part"
-F 5 "" H 5750 5000 50  0001 C CNN "PartNo"
+F 5 "963-EMF212B7104KGHT " H 5750 5000 50  0001 C CNN "PartNo"
 F 6 "Mouser" H 5750 5000 50  0001 C CNN "Supplier"
 	1    5750 5000
@@
 F 3 "http://www.ti.com/lit/ds/symlink/sn65hvd72.pdf?HQS=TI-null-null-mousermode-df-pf-null-wwe&ts=1590747515592" H 2500 3900 50  0001 C CNN
 F 4 "Mouser" H 2500 3900 50  0001 C CNN "Supplier"
+F 5 "595-SN65HVD72D" H 2500 3900 50  0001 C CNN "PartNo"
 	1    2500 3900
 	-1   0    0    -1
@@
 F 0 "C14" V 3629 3700 50  0000 C CNN
 F 1 "100n" V 3538 3700 50  0000 C CNN
-F 2 "Capacitor_SMD:C_0603_1608Metric_Pad1.05x0.95mm_HandSolder" H 3400 3700 50  0001 C CNN
+F 2 "Capacitor_SMD:C_0805_2012Metric_Pad1.15x1.40mm_HandSolder" H 3400 3700 50  0001 C CNN
 F 3 "~" H 3400 3700 50  0001 C CNN
 F 4 "" H 3400 3700 50  0001 C CNN "Part"
-F 5 "" H 3400 3700 50  0001 C CNN "PartNo"
+F 5 "963-EMF212B7104KGHT " H 3400 3700 50  0001 C CNN "PartNo"
 F 6 "Mouser" H 3400 3700 50  0001 C CNN "Supplier"
 	1    3400 3700
@@
 F 3 "https://www.mouser.de/datasheet/2/308/FAN3214T_F085-D-1805909.pdf" H 2800 6050 50  0001 C CNN
 F 4 "Mouser" H 2800 6050 50  0001 C CNN "Supplier"
+F 5 "512-FAN3214TMX" H 2800 6050 50  0001 C CNN "PartNo"
 	1    2800 6050
 	1    0    0    -1
@@
 F 3 "~" H 1300 6100 50  0001 C CNN
 F 4 "" H 1300 6100 50  0001 C CNN "Part"
-F 5 "" H 1300 6100 50  0001 C CNN "PartNo"
+F 5 "871-B41231A4109M000" H 1300 6100 50  0001 C CNN "PartNo"
 F 6 "Mouser" H 1300 6100 50  0001 C CNN "Supplier"
 	1    1300 6100
@@
 F 0 "C13" H 1942 5696 50  0000 L CNN
 F 1 "100n" V 1950 5450 50  0000 L CNN
-F 2 "Capacitor_SMD:C_0603_1608Metric_Pad1.05x0.95mm_HandSolder" H 1850 5650 50  0001 C CNN
+F 2 "Capacitor_SMD:C_0805_2012Metric_Pad1.15x1.40mm_HandSolder" H 1850 5650 50  0001 C CNN
 F 3 "~" H 1850 5650 50  0001 C CNN
 F 4 "" H 1850 5650 50  0001 C CNN "Part"
-F 5 "" H 1850 5650 50  0001 C CNN "PartNo"
+F 5 "963-EMF212B7104KGHT " H 1850 5650 50  0001 C CNN "PartNo"
 F 6 "Mouser" H 1850 5650 50  0001 C CNN "Supplier"
 	1    1850 5650
@@
 F 3 "~" H 9200 1150 50  0001 C CNN
 F 4 "" H 9200 1150 50  0001 C CNN "Part"
-F 5 "710-61300821121 " H 9200 1150 50  0001 C CNN "PartNo"
+F 5 "710-61300821121" H 9200 1150 50  0001 C CNN "PartNo"
 F 6 "Mouser" H 9200 1150 50  0001 C CNN "Supplier"
 	1    9200 1150
@@
 F 3 "~" H 9200 1800 50  0001 C CNN
 F 4 "" H 9200 1800 50  0001 C CNN "Part"
-F 5 "710-61300821121 " H 9200 1800 50  0001 C CNN "PartNo"
+F 5 "710-61300821121" H 9200 1800 50  0001 C CNN "PartNo"
 F 6 "Mouser" H 9200 1800 50  0001 C CNN "Supplier"
 	1    9200 1800
@@
 F 0 "C21" H 10915 3496 50  0000 L CNN
 F 1 "1n / 50V" H 10915 3405 50  0000 L CNN
-F 2 "Capacitor_SMD:C_0603_1608Metric_Pad1.05x0.95mm_HandSolder" H 10838 3300 50  0001 C CNN
+F 2 "Capacitor_SMD:C_0805_2012Metric_Pad1.15x1.40mm_HandSolder" H 10838 3300 50  0001 C CNN
 F 3 "~" H 10800 3450 50  0001 C CNN
 F 4 "" H 10800 3450 50  0001 C CNN "Part"
-F 5 "" H 10800 3450 50  0001 C CNN "PartNo"
+F 5 "77-VJ0805A102KXAAC" H 10800 3450 50  0001 C CNN "PartNo"
 F 6 "Mouser" H 10800 3450 50  0001 C CNN "Supplier"
 	1    10800 3450
@@
 F 0 "C16" V 10550 4700 50  0000 L CNN
 F 1 "100u / 6.3V" V 10750 4350 50  0000 L CNN
-F 2 "Capacitor_Tantalum_SMD:CP_EIA-7343-15_Kemet-W_Pad2.25x2.55mm_HandSolder" H 10650 4600 50  0001 C CNN
+F 2 "Capacitor_SMD:C_0805_2012Metric_Pad1.15x1.40mm_HandSolder" H 10650 4600 50  0001 C CNN
 F 3 "~" H 10650 4600 50  0001 C CNN
 F 4 "" H 10650 4600 50  0001 C CNN "Part"
-F 5 "" H 10650 4600 50  0001 C CNN "PartNo"
+F 5 "581-TLCR107M006RTA " H 10650 4600 50  0001 C CNN "PartNo"
 F 6 "Mouser" H 10650 4600 50  0001 C CNN "Supplier"
 	1    10650 4600
@@
 F 0 "C22" V 10850 4700 50  0000 L CNN
 F 1 "1u / 10V" V 11050 4450 50  0000 L CNN
-F 2 "Capacitor_SMD:C_0603_1608Metric_Pad1.05x0.95mm_HandSolder" H 10950 4600 50  0001 C CNN
+F 2 "Capacitor_SMD:C_0805_2012Metric_Pad1.15x1.40mm_HandSolder" H 10950 4600 50  0001 C CNN
 F 3 "~" H 10950 4600 50  0001 C CNN
 F 4 "" H 10950 4600 50  0001 C CNN "Part"
-F 5 "" H 10950 4600 50  0001 C CNN "PartNo"
+F 5 "77-VJ805Y105KXARW1BC " H 10950 4600 50  0001 C CNN "PartNo"
 F 6 "Mouser" H 10950 4600 50  0001 C CNN "Supplier"
 	1    10950 4600
@@
 F 3 "~" H 5750 1200 50  0001 C CNN
 F 4 "" H 5750 1200 50  0001 C CNN "Part"
-F 5 "710-61304011121 " H 5750 1200 50  0001 C CNN "PartNo"
+F 5 "710-61304011121" H 5750 1200 50  0001 C CNN "PartNo"
 F 6 "Mouser" H 5750 1200 50  0001 C CNN "Supplier"
 	1    5750 1200

Commit message: Finish Rev1 PCB Layout and send off to fab
PCB layout is done now, collect Revisions in REVISION.md
TODO updated with current tasks
Parts:
- added R36: Reset Pulldown, Resistor_SMD:R_0603_1608Metric_Pad1.05x0.95mm_HandSolder, symbol Device:R_Small
Changed lines of the file:
@@
 Wire Wire Line
 	6350 3650 6900 3650
-Wire Wire Line
-	6350 4400 7000 4400
 Text Label 7000 4400 2    50   ~ 0
 ATmega_RESET
@@
 Text Notes 5200 700  0    50   ~ 0
 ATmega UART2 Connector\n
+Wire Wire Line
+	6350 4400 7200 4400
+$Comp
+L Device:R_Small R36
+U 1 1 5EE08814
+P 7200 4500
+F 0 "R36" H 7259 4546 50  0000 L CNN
+F 1 "Reset Pulldown" H 7259 4455 50  0000 L CNN
+F 2 "Resistor_SMD:R_0603_1608Metric_Pad1.05x0.95mm_HandSolder" H 7200 4500 50  0001 C CNN
+F 3 "~" H 7200 4500 50  0001 C CNN
+	1    7200 4500
+	1    0    0    -1
+$EndComp
+$Comp
+L power:GND #PWR029
+U 1 1 5EE08CC5
+P 7200 4600
+F 0 "#PWR029" H 7200 4350 50  0001 C CNN
+F 1 "GND" H 7205 4427 50  0000 C CNN
+F 2 "" H 7200 4600 50  0001 C CNN
+F 3 "" H 7200 4600 50  0001 C CNN
+	1    7200 4600
+	1    0    0    -1
+$EndComp
 $EndSCHEMATC

Commit message: Update doc
Parts:
- removed J4: Conn_02x04_Top_Bottom, Connector_PinHeader_2.54mm:PinHeader_2x04_P2.54mm_Vertical, symbol Connector_Generic:Conn_02x04_Top_Bottom
- added J?: Conn_01x04, symbol Connector_Generic:Conn_01x04
- added R? (x3): 1k, symbol Device:R_Small
Connections:
- net labels added: ESP_IO15
- wire segments 170 -> 182
- no-connect marks 26 -> 25
Other:
- moved on the sheet: J5, R3, R4, R5, R6

Commit message: Testing build
Parts:
- C16: footprint Capacitor_SMD:C_0805_2012Metric_Pad1.15x1.40mm_HandSolder -> Capacitor_Tantalum_SMD:CP_EIA-2012-15_AVX-P_Pad1.30x1.05mm_HandSolder; symbol Device:C_Small -> Device:CP_Small
- gave numbers to parts that had none: 4
Changed lines of the file:
@@
 $Descr A4 11693 8268
 encoding utf-8
-Sheet 3 5
+Sheet 3 4
 Title "FGCCS-Ctrl22"
 Date "2020-08-11"
@@
 Connection ~ 10500 3200
 $Comp
-L Device:C_Small C16
+L Device:CP_Small C16
 U 1 1 5EC15E77
 P 10650 4600
 F 0 "C16" V 10550 4700 50  0000 L CNN
 F 1 "100u / 6.3V" V 10750 4350 50  0000 L CNN
-F 2 "Capacitor_SMD:C_0805_2012Metric_Pad1.15x1.40mm_HandSolder" H 10650 4600 50  0001 C CNN
+F 2 "Capacitor_Tantalum_SMD:CP_EIA-2012-15_AVX-P_Pad1.30x1.05mm_HandSolder" H 10650 4600 50  0001 C CNN
 F 3 "~" H 10650 4600 50  0001 C CNN
 F 4 "" H 10650 4600 50  0001 C CNN "Part"
@@
 ESP_IO15
 $Comp
-L Connector_Generic:Conn_01x04 J?
+L Connector_Generic:Conn_01x04 J4
 U 1 1 5F466074
 P 9300 1550
-F 0 "J?" H 9450 1350 50  0000 C CNN
+F 0 "J4" H 9450 1350 50  0000 C CNN
 F 1 "Conn_01x04" H 9600 1450 50  0000 C CNN
 F 2 "" H 9300 1550 50  0001 C CNN
@@
 Connection ~ 9100 750
 $Comp
-L Device:R_Small R?
+L Device:R_Small R34
 U 1 1 5F47B25C
 P 9400 900
-F 0 "R?" V 9350 1050 50  0000 C CNN
+F 0 "R34" V 9350 1050 50  0000 C CNN
 F 1 "1k" V 9295 900 50  0000 C CNN
 F 2 "" H 9400 900 50  0001 C CNN
@@
 $EndComp
 $Comp
-L Device:R_Small R?
+L Device:R_Small R37
 U 1 1 5F47BC59
 P 9400 1100
-F 0 "R?" V 9350 1250 50  0000 C CNN
+F 0 "R37" V 9350 1250 50  0000 C CNN
 F 1 "1k" V 9295 1100 50  0000 C CNN
 F 2 "" H 9400 1100 50  0001 C CNN
@@
 $EndComp
 $Comp
-L Device:R_Small R?
+L Device:R_Small R38
 U 1 1 5F47BE53
 P 9400 1300
-F 0 "R?" V 9350 1450 50  0000 C CNN
+F 0 "R38" V 9350 1450 50  0000 C CNN
 F 1 "1k" V 9295 1300 50  0000 C CNN
 F 2 "" H 9400 1300 50  0001 C CNN

Commit message: Finish Revision 1.1 layout
Parts:
- removed R36: Reset Pulldown, Resistor_SMD:R_0603_1608Metric_Pad1.05x0.95mm_HandSolder, symbol Device:R_Small
- J3: footprint Connector_PinHeader_2.54mm:PinHeader_1x04_P2.54mm_Vertical -> atmevse-footprints:UART2-Header
- J4: footprint (none) -> atmevse-footprints:UART0-Header
- J5: footprint Connector_PinHeader_2.54mm:PinHeader_2x04_P2.54mm_Vertical -> atmevse-footprints:PROGRAM-Header
- R34, R37, R38: footprint (none) -> Resistor_SMD:R_0603_1608Metric_Pad1.05x0.95mm_HandSolder
Changed lines of the file:
@@
 Wire Wire Line
 	6350 3650 6900 3650
-Text Label 7000 4400 2    50   ~ 0
+Text Label 6900 4400 2    50   ~ 0
 ATmega_RESET
 Text Label 6900 3500 2    50   ~ 0
@@
 F 0 "J5" H 9150 1800 50  0000 C CNN
 F 1 "Conn_02x04_Top_Bottom" H 9150 2326 50  0000 C CNN
-F 2 "Connector_PinHeader_2.54mm:PinHeader_2x04_P2.54mm_Vertical" H 9100 2100 50  0001 C CNN
+F 2 "atmevse-footprints:PROGRAM-Header" H 9100 2100 50  0001 C CNN
 F 3 "~" H 9100 2100 50  0001 C CNN
 F 4 "" H 9100 2100 50  0001 C CNN "Part"
@@
 F 0 "J3" H 5830 1192 50  0000 L CNN
 F 1 "Conn_01x04" H 5830 1101 50  0000 L CNN
-F 2 "Connector_PinHeader_2.54mm:PinHeader_1x04_P2.54mm_Vertical" H 5750 1200 50  0001 C CNN
+F 2 "atmevse-footprints:UART2-Header" H 5750 1200 50  0001 C CNN
 F 3 "~" H 5750 1200 50  0001 C CNN
 F 4 "" H 5750 1200 50  0001 C CNN "Part"
@@
 ATmega UART2 Connector\n
 Wire Wire Line
-	6350 4400 7200 4400
-$Comp
-L Device:R_Small R36
-U 1 1 5EE08814
-P 7200 4500
-F 0 "R36" H 7259 4546 50  0000 L CNN
-F 1 "Reset Pulldown" H 7259 4455 50  0000 L CNN
-F 2 "Resistor_SMD:R_0603_1608Metric_Pad1.05x0.95mm_HandSolder" H 7200 4500 50  0001 C CNN
-F 3 "~" H 7200 4500 50  0001 C CNN
-	1    7200 4500
-	1    0    0    -1
-$EndComp
-$Comp
-L power:GND #PWR029
-U 1 1 5EE08CC5
-P 7200 4600
-F 0 "#PWR029" H 7200 4350 50  0001 C CNN
-F 1 "GND" H 7205 4427 50  0000 C CNN
-F 2 "" H 7200 4600 50  0001 C CNN
-F 3 "" H 7200 4600 50  0001 C CNN
-	1    7200 4600
-	1    0    0    -1
-$EndComp
-Wire Wire Line
 	650  5750 650  5950
 Wire Wire Line
@@
 F 0 "J4" H 9450 1350 50  0000 C CNN
 F 1 "Conn_01x04" H 9600 1450 50  0000 C CNN
-F 2 "" H 9300 1550 50  0001 C CNN
+F 2 "atmevse-footprints:UART0-Header" H 9300 1550 50  0001 C CNN
 F 3 "~" H 9300 1550 50  0001 C CNN
 	1    9300 1550
@@
 F 0 "R34" V 9350 1050 50  0000 C CNN
 F 1 "1k" V 9295 900 50  0000 C CNN
-F 2 "" H 9400 900 50  0001 C CNN
+F 2 "Resistor_SMD:R_0603_1608Metric_Pad1.05x0.95mm_HandSolder" H 9400 900 50  0001 C CNN
 F 3 "~" H 9400 900 50  0001 C CNN
 	1    9400 900
@@
 F 0 "R37" V 9350 1250 50  0000 C CNN
 F 1 "1k" V 9295 1100 50  0000 C CNN
-F 2 "" H 9400 1100 50  0001 C CNN
+F 2 "Resistor_SMD:R_0603_1608Metric_Pad1.05x0.95mm_HandSolder" H 9400 1100 50  0001 C CNN
 F 3 "~" H 9400 1100 50  0001 C CNN
 	1    9400 1100
@@
 F 0 "R38" V 9350 1450 50  0000 C CNN
 F 1 "1k" V 9295 1300 50  0000 C CNN
-F 2 "" H 9400 1300 50  0001 C CNN
+F 2 "Resistor_SMD:R_0603_1608Metric_Pad1.05x0.95mm_HandSolder" H 9400 1300 50  0001 C CNN
 F 3 "~" H 9400 1300 50  0001 C CNN
 	1    9400 1300
@@
 Wire Wire Line
 	9700 2200 9400 2200
+Wire Wire Line
+	6350 4400 6900 4400
 $EndSCHEMATC
